File: hardware/USBcablecracker.sch (KiCad schematic (older format))
At the start: 56 parts, among them P1 USB_A, P10 USB_A, P11 USB_B, P12 CONN_01X09, P2 CONN_01X02, P3 USB_B-Micro, P6 CONN_01X09, P7 USB_B-Mini, P8 USB_B-Micro-3.0, P9 USB_TYPEC-S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

Commit message: Modify PCB to v2.0, delete switch, add an analog switch and a button instead.
Parts:
- removed C8: 22uF, Capacitors_Tantalum_SMD:Tantalum_Case-A_EIA-3216-18_Wave, symbol CP_Small
- removed R9: 10K, Resistors_SMD:R_0603_HandSoldering, symbol R_Small
- removed SW1: Switch_SPDT_x2, USBcablecracker:DPDT, symbol Switch_SPDT_x2
- added C14, C15: 100nF, Capacitors_SMD:C_0603_HandSoldering, symbol C_Small
- added C8: 10uF, Capacitors_SMD:C_0603_HandSoldering, symbol C_Small
- added Q1, Q2, Q3: CJ2302, TO_SOT_Packages_SMD:SOT-23_Handsoldering, symbol Q_NMOS_GSD
- added R23: 1K, Resistors_SMD:R_0603_HandSoldering, symbol R_Small
- added R24: 33, Resistors_SMD:R_0603_HandSoldering, symbol R_Small
- added R26: 10k, Resistors_SMD:R_0603_HandSoldering, symbol R_Small
- added SW1: SW_SPST, Buttons_Switches_SMD:SW_SPST_EVQP0, symbol SW_SPST
- added U4: SN74LVC1G3157, TO_SOT_Packages_SMD:SOT-23-6_Handsoldering, symbol NC7SB3157
- added U5: 4053, Housings_SSOP:TSSOP-16_4.4x5mm_Pitch0.65mm, symbol 4053
- DS1: footprint Display:WC1602A -> USBcablecracker:WC1602A
- P1, P10, P11: symbol USB_A -> USB_A-RESCUE-USBcablecracker
- U3: symbol AD620 -> AD620-RESCUE-USBcablecracker
Connections:
- net labels added: AX, AY, SELECT
- net labels removed: TEST5, TEST6
- wire segments 220 -> 245
- no-connect marks 10 -> 37
Other:
- note added: "Vref=2.56V"
- moved on the sheet: C1, C10, C12, C5, C6, C7, CONN1, D1, D2, D3, D4, P2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
